File: PCB Entwurf/humidity-control/humidity-control/humidity-control.kicad_pcb (KiCad board)
At the start: 2 copper layers, 10 parts

Commit message: Remove, modificationa in files and also added new file
Parts:
- removed the ? at (169.0, 68.0)
- removed the ? at (169.0, 71.0)
- removed the ? at (169.0, 74.0)
- added ?: , , F.Cu at (157.5, 86.2)
- added ?: , , F.Cu at (157.6, 81.1)
- added L7805C: TO-220-3_Vertical, Package_TO_SOT_THT:TO-220-3_Vertical, F.Cu at (143.0, 77.0)
- moved ? 22.9 mm to (157.6, 101.4)
- moved ULN7002A 22.8 mm to (136.3, 86.1)
- moved HDT11 22.1 mm to (125.0, 89.7)
- moved ? 20.7 mm to (157.6, 96.3)
- moved ? 18.6 mm to (157.6, 91.2)
- moved Diode 17.7 mm to (150.1, 94.8)
- moved ? 15.9 mm to (157.6, 76.0)
- renumbered REF** to Diode
Routing:
- net (no net): track 339.0 -> 316.7 mm
Other:
- board text removed: "+5V"
